Commit message: fixed redifing global symbol: pi

File: kuka_arm_description/urdf/kr210.urdf.xacro (robot description, xacro)
@@ -2,5 +2,4 @@
 <robot name="kuka_arm" xmlns:xacro="http://www.ros.org/wiki/xacro">
   <!--Define constants-->
-  <xacro:property name="pi" value="3.141592654"/>
   <xacro:property name="deg" value="0.017453293"/><!--degrees to radians-->
   <xacro:property name="mass0" value="150" />

Commit message: set z=0 for world_joint

File: kuka_arm_description/urdf/kr210.urdf.xacro (robot description, xacro)
@@ -309,5 +309,5 @@
     <parent link="world"/>
     <child link="base_link"/>
-    <origin xyz="0 0 0.25" rpy="0 0 0"/>
+    <origin xyz="0 0 0" rpy="0 0 0"/>
   </joint>
   <!--<joint name="fixed_base_joint" type="fixed">
